File: pcb_design/usb-to-uart/usb-to-uart.kicad_pcb (KiCad board)
At the start: 2 copper layers, 18 parts, among them IC1 CP2102, J1 Conn_01x06_Male, J2 USB_C_Receptacle_USB2.0, J3 Conn_01x04_Male, J4 Conn_01x04_Male, Q1 2N2219, SW1 SW_MEC_5G

Commit message: routing 1 completed
Parts:
- removed IC1: CP2102, CP2102:QFN50P500X500X100-29N
- removed Q1: 2N2219, Package_TO_SOT_THT:TO-39-3
- added CP2102: CP2102, CP2102:QFN50P500X500X100-29N, F.Cu at (127.7, 73.8)
- added IC2: L8050QLT1G, npn_smd:L8050QLT1G, F.Cu at (140.0, 73.7)
- J2: value USB_C_Receptacle_USB2.0 -> TYPE-C-31-M-12; footprint Connector_USB:USB_C_Receptacle_GCT_USB4135-GF-A_6P_TopMnt_Horizontal -> usb c:HRO_TYPE-C-31-M-12
- moved SW1 179.9 mm to (112.4, 68.4), turned to -90 degrees
- moved C1 179.6 mm to (122.0, 75.4)
- moved C2 176.3 mm to (126.0, 78.4)
- moved R1 172.2 mm to (133.2, 77.4)
- moved R4 162.8 mm to (120.2, 79.7)
- moved J2 162.3 mm to (109.3, 78.0), turned to -90 degrees
- moved J4 158.8 mm to (137.2, 81.8)
- moved C3 156.6 mm to (146.2, 82.4)
- moved R3 152.3 mm to (116.4, 74.2), turned to 90 degrees
- moved R2 148.8 mm to (128.9, 80.6)
- moved R5 141.9 mm to (136.4, 72.8), turned to -90 degrees
- moved R7 129.9 mm to (145.7, 73.9), turned to 180 degrees
- moved J1 128.4 mm to (153.8, 74.0), turned to -90 degrees
- moved J3 127.9 mm to (137.4, 66.4)
- moved R6 122.2 mm to (146.2, 79.0)
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Connections:
- J1 pad 1: RTS -> 5V
- J1 pad 2: TXD -> DTR
- J1 pad 3: RXD -> TXD
- J1 pad 4: 5V -> RXD
- J1 pad 5: DTR -> GND
- J1 pad 6: GND -> RTS
- J3 pad 1: RI -> 3V3
- J3 pad 2: DCD -> RI
- J3 pad 3: SUSPEND -> DCD
- J4 pad 1: CTS -> GND
- J4 pad 2: GND -> SUSPEND
- J4 pad 4: 3V3 -> CTS
Routing:
- net GND: track 0.00 -> 140.2 mm, vias 0 -> 7
- net 5V: track 0.00 -> 80.9 mm, vias 0 -> 4
- net EN: track 0.00 -> 65.5 mm, vias 0 -> 2
- net 3V3: track 0.00 -> 59.1 mm, vias 0 -> 5
- net DTR: track 0.00 -> 49.4 mm, vias 0 -> 4
- net RTS: track 0.00 -> 34.7 mm, vias 0 -> 2
- net RXD: track 0.00 -> 29.9 mm
- net TXD: track 0.00 -> 29.5 mm
- net RI: track 0.00 -> 19.0 mm, vias 0 -> 2
- net CTS: track 0.00 -> 17.6 mm
- net DCD: track 0.00 -> 17.3 mm
- net DSR: track 0.00 -> 17.2 mm
- net D+: track 0.00 -> 16.5 mm, vias 0 -> 2
- net D-: track 0.00 -> 15.6 mm
- net SUSPEND: track 0.00 -> 10.4 mm
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- added copper zone on B.Cu, net GND
Other:
- board outline added: 50 x 20 mm

Commit message: PCB Completed
Parts:
- removed CP2102: CP2102, CP2102:QFN50P500X500X100-29N
- added IC1: CP2102, CP2102:QFN50P500X500X100-29N, F.Cu at (137.0, 109.3)
- moved C1 42.0 mm to (142.4, 112.1)
- moved R7 41.7 mm to (145.7, 115.6)
- moved R3 37.6 mm to (130.0, 109.3), turned to 0 degrees
- moved R4 36.9 mm to (129.8, 115.3)
- moved C2 36.0 mm to (142.4, 110.5)
- moved IC2 36.0 mm to (147.7, 108.8), turned to -90 degrees
- moved SW1 35.8 mm to (121.7, 103.0), turned to 90 degrees
- moved J3 35.5 mm to (138.3, 101.9)
- moved J2 34.9 mm to (119.8, 111.3)
- moved J1 34.5 mm to (152.2, 108.5)
- moved D1 34.3 mm to (142.4, 105.9)
- moved J4 33.5 mm to (138.3, 115.3)
- moved R2 31.8 mm to (130.0, 112.4)
- moved R5 30.6 mm to (145.7, 102.0), turned to 0 degrees
- moved R1 30.4 mm to (130.0, 107.6)
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Connections:
- J1 pad 2: DTR -> DSR
- J1 pad 5: GND -> EN
- J1 pad 6: RTS -> GND
- J3 pad 4: DSR -> DTR
- J4 pad 3: EN -> CTS
- J4 pad 4: CTS -> RTS
Routing:
- net GND: track 140.2 -> 55.4 mm, vias 7 -> 3
- net 3V3: track 59.1 -> 18.0 mm, vias 5 -> 2
- net DTR: track 49.4 -> 12.4 mm, vias 4 -> 0
- net 5V: track 80.9 -> 45.8 mm
- net RTS: track 34.7 -> 22.6 mm, vias 2 -> 1
- net Net-(D1-Pad2): track 2.75 -> 13.5 mm, vias 0 -> 2
- net TXD: track 29.5 -> 18.9 mm
- net RI: track 19.0 -> 8.42 mm, vias 2 -> 0
- net RXD: track 29.9 -> 19.4 mm
- net Net-(C1-Pad2): track 2.78 -> 13.1 mm, vias 0 -> 2
- net Net-(IC1-Pad11): track 7.36 -> 16.9 mm
- net DCD: track 17.3 -> 8.59 mm
- net SUSPEND: track 10.4 -> 3.82 mm
- net Net-(IC2-Pad1): track 3.10 -> 8.33 mm, vias 0 -> 2
- net CTS: track 17.6 -> 12.6 mm
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Other:
- board size 50 x 20 mm -> 38.2 x 17 mm
