File: pcb_design/usb-to-uart/usb-to-uart.kicad_sch (KiCad schematic)
At the start: 4 parts

Commit message: completed schematic design
Parts:
- added C1: 0.1uF, Capacitor_SMD:C_0603_1608Metric, symbol Device:C
- added C2, C3: 1uF, Capacitor_SMD:C_0201_0603Metric, symbol Device:C
- added D1: LED, symbol Device:LED
- added J3, J4: Conn_01x04_Male, symbol Connector:Conn_01x04_Male
- added Q1: 2N2219, Package_TO_SOT_THT:TO-39-3, symbol Transistor_BJT:2N2219
- added R2, R5, R6: 10K, symbol Device:R
- added R3, R4, R7: 5.1K, symbol Device:R
- added SW1: SW_MEC_5G, symbol Switch:SW_MEC_5G
- J2: renamed from J?; footprint (none) -> Connector_USB:USB_C_Receptacle_GCT_USB4135-GF-A_6P_TopMnt_Horizontal
- gave numbers to parts that had none: 3
Connections:
- net DTR: now also R5.1
- net GND: now also J1.6 (Pin_6), J2.S1 (SHIELD), C1.1, C2.2, C3.2, D1.1 (K), J4.2 (Pin_2), R3.2, R4.2, SW1.1 (A), SW1.2 (A)
- net RTS: now also Q1.1 (E)
- net DCD: now reaches IC1.1 (DCD)
- net DCD: now also J3.2 (Pin_2)
- net SUSPEND: now reaches IC1.12 (SUSPEND)
- net SUSPEND: now also J3.3 (Pin_3)
- net RI: now reaches IC1.2 (RI)
- net RI: now also J3.1 (Pin_1)
- net CTS: now reaches IC1.23 (CTS)
- net CTS: now also J4.1 (Pin_1)
- net DSR: now reaches IC1.27 (DSR)
- net DSR: now also J3.4 (Pin_4)
- net at IC1.6 (VDD): now also C1.2
- net +5V: now reaches IC1.7 (REGIN)
- net +5V: now also IC1.8 (VBUS), J1.4 (Pin_4), J2.A4 (VBUS), J2.A9 (VBUS), J2.B4 (VBUS), J2.B9 (VBUS), C2.1, R7.1
- net at IC1.9 (~{RST}): now also R2.1
- net at J2.A5 (CC1): now also R3.1
- net at J2.B5 (CC2): now also R4.1
- new net: Q1.2 (B), R5.2
- new net: D1.2 (A), R7.2
- new net +3.3V: J4.4 (Pin_4), R2.2, R6.2
- new net EN: C3.1, J4.3 (Pin_3), Q1.3 (C), R6.1, SW1.3 (B), SW1.4 (B)
- no-connect marks 11 -> 13
Other:
- note added: "CONNECTORS"
- note added: "SWITCH"
- moved on the sheet: J1, J2

Commit message: footprint assignment done
Parts:
- C2, C3: footprint Capacitor_SMD:C_0201_0603Metric -> Capacitor_SMD:C_0603_1608Metric
- D1, R1, R2, R3, R4, R5, R6, R7: footprint (none) -> LED_SMD:LED_0603_1608Metric
- IC1: footprint QFN50P500X500X100-29N-D -> CP2102:QFN50P500X500X100-29N
- J1: footprint (none) -> Pin header 01x06:TE_825433-6
- J3, J4: footprint (none) -> Pin header 01x04:61300411121
- SW1: footprint (none) -> Tactile Switch:SW_TL3305AF260QG
Changed lines of the file:
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@@
     (property "Reference" "IC1" (id 0) (at 62.23 68.3512 0))
     (property "Value" "CP2102" (id 1) (at 62.23 70.8912 0))
-    (property "Footprint" "QFN50P500X500X100-29N-D" (id 2) (at 58.42 62.23 0)
+    (property "Footprint" "CP2102:QFN50P500X500X100-29N" (id 2) (at 58.42 62.23 0)
       (effects (font (size 1.27 1.27)) (justify left) hide)
     )
@@
       (effects (font (size 1 1)) (justify left))
     )
-    (property "Footprint" "Capacitor_SMD:C_0201_0603Metric" (id 2) (at 30.1752 121.92 0)
+    (property "Footprint" "Capacitor_SMD:C_0603_1608Metric" (id 2) (at 30.1752 121.92 0)
       (effects (font (size 1.27 1.27)) hide)
     )
@@
     (property "Reference" "J4" (id 0) (at 127.635 157.48 0))
     (property "Value" "Conn_01x04_Male" (id 1) (at 127.635 160.02 0))
-    (property "Footprint" "" (id 2) (at 127 165.1 0)
+    (property "Footprint" "Pin header 01x04:61300411121" (id 2) (at 127 165.1 0)
       (effects (font (size 1.27 1.27)) hide)
     )
@@
     (property "Reference" "J3" (id 0) (at 85.725 157.48 0))
     (property "Value" "Conn_01x04_Male" (id 1) (at 85.725 160.02 0))
-    (property "Footprint" "" (id 2) (at 85.09 165.1 0)
+    (property "Footprint" "Pin header 01x04:61300411121" (id 2) (at 85.09 165.1 0)
       (effects (font (size 1.27 1.27)) hide)
     )
@@
     (property "Reference" "D1" (id 0) (at 269.5575 52.07 0))
     (property "Value" "LED" (id 1) (at 269.5575 54.61 0))
-    (property "Footprint" "" (id 2) (at 267.97 59.69 0)
+    (property "Footprint" "LED_SMD:LED_0603_1608Metric" (id 2) (at 267.97 59.69 0)
       (effects (font (size 1.27 1.27)) hide)
     )
@@
       (effects (font (size 1 1)))
     )
-    (property "Footprint" "" (id 2) (at 217.678 63.5 90)
+    (property "Footprint" "LED_SMD:LED_0603_1608Metric" (id 2) (at 217.678 63.5 90)
       (effects (font (size 1.27 1.27)) hide)
     )
@@
     (property "Reference" "J1" (id 0) (at 34.925 156.21 0))
     (property "Value" "Conn_01x06_Male" (id 1) (at 34.925 158.75 0))
-    (property "Footprint" "" (id 2) (at 34.29 166.37 0)
+    (property "Footprint" "Pin header 01x06:TE_825433-6" (id 2) (at 34.29 166.37 0)
       (effects (font (size 1.27 1.27)) hide)
     )
@@
       (effects (font (size 1 1)) (justify left))
     )
-    (property "Footprint" "" (id 2) (at 37.592 114.3 90)
+    (property "Footprint" "LED_SMD:LED_0603_1608Metric" (id 2) (at 37.592 114.3 90)
       (effects (font (size 1.27 1.27)) hide)
     )
@@
       (effects (font (size 1 1)) (justify left))
     )
-    (property "Footprint" "" (id 2) (at 42.672 114.3 90)
+    (property "Footprint" "LED_SMD:LED_0603_1608Metric" (id 2) (at 42.672 114.3 90)
       (effects (font (size 1.27 1.27)) hide)
     )
@@
       (effects (font (size 1 1)) (justify left))
     )
-    (property "Footprint" "Capacitor_SMD:C_0201_0603Metric" (id 2) (at 216.8652 76.2 0)
+    (property "Footprint" "Capacitor_SMD:C_0603_1608Metric" (id 2) (at 216.8652 76.2 0)
       (effects (font (size 1.27 1.27)) hide)
     )
@@
       (effects (font (size 1 1)))
     )
-    (property "Footprint" "" (id 2) (at 196.85 83.058 90)
+    (property "Footprint" "LED_SMD:LED_0603_1608Metric" (id 2) (at 196.85 83.058 90)
       (effects (font (size 1.27 1.27)) hide)
     )
@@
       (effects (font (size 1 1)))
     )
-    (property "Footprint" "" (id 2) (at 143.51 75.438 90)
+    (property "Footprint" "LED_SMD:LED_0603_1608Metric" (id 2) (at 143.51 75.438 90)
       (effects (font (size 1.27 1.27)) hide)
     )
@@
       (effects (font (size 1 1)))
     )
-    (property "Footprint" "" (id 2) (at 143.51 77.978 90)
+    (property "Footprint" "LED_SMD:LED_0603_1608Metric" (id 2) (at 143.51 77.978 90)
       (effects (font (size 1.27 1.27)) hide)
     )
@@
       (effects (font (size 1 1)))
     )
-    (property "Footprint" "" (id 2) (at 256.54 61.468 90)
+    (property "Footprint" "LED_SMD:LED_0603_1608Metric" (id 2) (at 256.54 61.468 90)
       (effects (font (size 1.27 1.27)) hide)
     )
@@
     (property "Reference" "SW1" (id 0) (at 201.93 60.96 0))
     (property "Value" "SW_MEC_5G" (id 1) (at 201.93 63.5 0))
-    (property "Footprint" "" (id 2) (at 201.93 63.5 0)
+    (property "Footprint" "Tactile Switch:SW_TL3305AF260QG" (id 2) (at 201.93 63.5 0)
       (effects (font (size 1.27 1.27)) hide)
     )
@@
     )
     (path "/2257ec34-a663-45b3-a032-916ae0648610"
-      (reference "C2") (unit 1) (value "1uF") (footprint "Capacitor_SMD:C_0201_0603Metric")
+      (reference "C2") (unit 1) (value "1uF") (footprint "Capacitor_SMD:C_0603_1608Metric")
     )
     (path "/a5596501-db2a-42ca-948d-b14422c03242"
-      (reference "C3") (unit 1) (value "1uF") (footprint "Capacitor_SMD:C_0201_0603Metric")
+      (reference "C3") (unit 1) (value "1uF") (footprint "Capacitor_SMD:C_0603_1608Metric")
     )
     (path "/4ae39f27-2944-4284-bca8-64562643e20d"
-      (reference "D1") (unit 1) (value "LED") (footprint "")
+      (reference "D1") (unit 1) (value "LED") (footprint "LED_SMD:LED_0603_1608Metric")
     )
     (path "/19e1cfca-f42e-485a-aa53-1eca42a8a91d"
-      (reference "IC1") (unit 1) (value "CP2102") (footprint "QFN50P500X500X100-29N-D")
+      (reference "IC1") (unit 1) (value "CP2102") (footprint "CP2102:QFN50P500X500X100-29N")
     )
     (path "/4d17ad65-4fed-4e16-a43b-1c88dfdd6512"
-      (reference "J1") (unit 1) (value "Conn_01x06_Male") (footprint "")
+      (reference "J1") (unit 1) (value "Conn_01x06_Male") (footprint "Pin header 01x06:TE_825433-6")
     )
     (path "/6f1388ec-3d70-4ef0-ab82-a5ad7120dc0f"
@@
     )
     (path "/4100ff93-7322-48cd-b43c-f7431896ea03"
-      (reference "J3") (unit 1) (value "Conn_01x04_Male") (footprint "")
+      (reference "J3") (unit 1) (value "Conn_01x04_Male") (footprint "Pin header 01x04:61300411121")
     )
     (path "/3d1f7290-de45-4d2d-9852-08ded667f3bb"
-      (reference "J4") (unit 1) (value "Conn_01x04_Male") (footprint "")
+      (reference "J4") (unit 1) (value "Conn_01x04_Male") (footprint "Pin header 01x04:61300411121")
     )
     (path "/153cfd11-638d-4c7e-8357-0d6cc66221d8"
@@
     )
     (path "/64e8e927-575a-4c2c-a206-bda209a97f88"
-      (reference "R1") (unit 1) (value "10K") (footprint "")
+      (reference "R1") (unit 1) (value "10K") (footprint "LED_SMD:LED_0603_1608Metric")
     )
     (path "/5c3f1a0a-5d2a-40ce-867f-cd84ce04da00"
-      (reference "R2") (unit 1) (value "10K") (footprint "")
+      (reference "R2") (unit 1) (value "10K") (footprint "LED_SMD:LED_0603_1608Metric")
     )
     (path "/be88c070-22ce-4508-b5f6-2df69a30e6fb"
-      (reference "R3") (unit 1) (value "5.1K") (footprint "")
+      (reference "R3") (unit 1) (value "5.1K") (footprint "LED_SMD:LED_0603_1608Metric")
     )
     (path "/c9e6c986-e0a6-47a7-ae07-6e75c90fa30d"
-      (reference "R4") (unit 1) (value "5.1K") (footprint "")
+      (reference "R4") (unit 1) (value "5.1K") (footprint "LED_SMD:LED_0603_1608Metric")
     )
     (path "/b550aefa-d800-464c-9635-bf17f66c318a"
-      (reference "R5") (unit 1) (value "10K") (footprint "")
+      (reference "R5") (unit 1) (value "10K") (footprint "LED_SMD:LED_0603_1608Metric")
     )
     (path "/4d154e2a-db48-4f01-a526-c5f1bdaabe04"
-      (reference "R6") (unit 1) (value "10K") (footprint "")
+      (reference "R6") (unit 1) (value "10K") (footprint "LED_SMD:LED_0603_1608Metric")
     )
     (path "/f0f63267-0887-4327-88c9-380f89b6f5dc"
-      (reference "R7") (unit 1) (value "5.1K") (footprint "")
+      (reference "R7") (unit 1) (value "5.1K") (footprint "LED_SMD:LED_0603_1608Metric")
     )
     (path "/f91b47af-0d41-4687-9b18-8f35940da2cc"
-      (reference "SW1") (unit 1) (value "SW_MEC_5G") (footprint "")
-    )
-  )
+      (reference "SW1") (unit 1) (value "SW_MEC_5G") (footprint "Tactile Switch:SW_TL3305AF260QG")
+    )
+  )

Commit message: routing 1 completed
Parts:
- removed J2: USB_C_Receptacle_USB2.0, Connector_USB:USB_C_Receptacle_GCT_USB4135-GF-A_6P_TopMnt_Horizontal, symbol Connector:USB_C_Receptacle_USB2.0
- removed Q1: 2N2219, Package_TO_SOT_THT:TO-39-3, symbol Transistor_BJT:2N2219
- added IC2: L8050QLT1G, npn_smd:L8050QLT1G, symbol L8050QLT1G:L8050QLT1G
- added J2: TYPE-C-31-M-12, usb c:HRO_TYPE-C-31-M-12, symbol TYPE-C-31-M-12:TYPE-C-31-M-12
Connections:
- net +3.3V: now also J3.1 (Pin_1); no longer J4.4 (Pin_4)
- net +5V: now also J1.1 (Pin_1), J2.A4B9 (VBUS), J2.B4A9 (VBUS); no longer J1.4 (Pin_4)
- net CTS: now also J4.4 (Pin_4); no longer J4.1 (Pin_1)
- net D+: now also J2.A6 (DP1), J2.B6 (DP2)
- net D-: now also J2.A7 (DN1), J2.B7 (DN2)
- net DCD: now also J3.3 (Pin_3); no longer J3.2 (Pin_2)
- net DTR: now also J1.2 (Pin_2); no longer J1.5 (Pin_5)
- net EN: now also IC2.3 (C)
- net GND: now also J1.5 (Pin_5), J4.1 (Pin_1), J2.A1B12 (GND), J2.B1A12 (GND), J2.S1 (SHIELD), J2.S2 (SHIELD), J2.S3 (SHIELD), J2.S4 (SHIELD); no longer J1.6 (Pin_6), J4.2 (Pin_2)
- net RI: now also J3.2 (Pin_2); no longer J3.1 (Pin_1)
- net RTS: now also J1.6 (Pin_6), IC2.2 (E); no longer J1.1 (Pin_1)
- net RXD: now also J1.4 (Pin_4); no longer J1.3 (Pin_3)
- net SUSPEND: now also J4.2 (Pin_2); no longer J3.3 (Pin_3)
- net TXD: now also J1.3 (Pin_3); no longer J1.2 (Pin_2)
- net at R5.2: now also IC2.1 (B)
- net at R3.1: now also J2.A5 (CC1)
- net at R4.1: now also J2.B5 (CC2)

Commit message: PCB Completed
Connections:
- net CTS: now also J4.3 (Pin_3); no longer J4.4 (Pin_4)
- net DSR: now also J1.2 (Pin_2); no longer J3.4 (Pin_4)
- net DTR: now also J3.4 (Pin_4); no longer J1.2 (Pin_2)
- net EN: now also J1.5 (Pin_5); no longer J4.3 (Pin_3)
- net GND: now also J1.6 (Pin_6); no longer J1.5 (Pin_5)
- net RTS: now also J4.4 (Pin_4); no longer J1.6 (Pin_6)
Changed lines of the file:
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@@
     )
   )
-  (global_label "GND" (shape input) (at 46.99 171.45 0) (fields_autoplaced)
-    (effects (font (size 1 1) bold) (justify left))
-    (property "Intersheet References" "${INTERSHEET_REFS}" (id 0) (at 52.0876 171.35 0)
+  (global_label "EN" (shape input) (at 46.99 171.45 0) (fields_autoplaced)
+    (effects (font (size 1 1) bold) (justify left))
+    (property "Intersheet References" "${INTERSHEET_REFS}" (id 0) (at 50.9924 171.35 0)
       (effects (font (size 1 1) bold) (justify left) hide)
     )
@@
     )
   )
-  (global_label "EN" (shape input) (at 137.16 167.64 0) (fields_autoplaced)
+  (global_label "CTS" (shape input) (at 137.16 167.64 0) (fields_autoplaced)
     (effects (font (size 1.27 1.27)) (justify left))
-    (property "Intersheet References" "${INTERSHEET_REFS}" (id 0) (at 142.0526 167.5606 0)
+    (property "Intersheet References" "${INTERSHEET_REFS}" (id 0) (at 143.0202 167.5606 0)
       (effects (font (size 1.27 1.27)) (justify left) hide)
     )
@@
     )
   )
-  (global_label "DTR" (shape input) (at 46.99 163.83 0) (fields_autoplaced)
-    (effects (font (size 1 1) bold) (justify left))
-    (property "Intersheet References" "${INTERSHEET_REFS}" (id 0) (at 51.8019 163.73 0)
-      (effects (font (size 1 1) bold) (justify left) hide)
-    )
-  )
-  (global_label "RTS" (shape input) (at 46.99 173.99 0) (fields_autoplaced)
-    (effects (font (size 1 1) bold) (justify left))
-    (property "Intersheet References" "${INTERSHEET_REFS}" (id 0) (at 51.7543 173.89 0)
+  (global_label "DSR" (shape input) (at 46.99 163.83 0) (fields_autoplaced)
+    (effects (font (size 1 1) bold) (justify left))
+    (property "Intersheet References" "${INTERSHEET_REFS}" (id 0) (at 51.9924 163.73 0)
+      (effects (font (size 1 1) bold) (justify left) hide)
+    )
+  )
+  (global_label "GND" (shape input) (at 46.99 173.99 0) (fields_autoplaced)
+    (effects (font (size 1 1) bold) (justify left))
+    (property "Intersheet References" "${INTERSHEET_REFS}" (id 0) (at 52.0876 173.89 0)
       (effects (font (size 1 1) bold) (justify left) hide)
     )
@@
     )
   )
-  (global_label "CTS" (shape input) (at 137.16 170.18 0) (fields_autoplaced)
+  (global_label "RTS" (shape input) (at 137.16 170.18 0) (fields_autoplaced)
     (effects (font (size 1 1)) (justify left))
     (property "Intersheet References" "${INTERSHEET_REFS}" (id 0) (at 141.7743 170.1175 0)
@@
     )
   )
-  (global_label "DSR" (shape input) (at 93.98 170.18 0) (fields_autoplaced)
-    (effects (font (size 1 1)) (justify left))
-    (property "Intersheet References" "${INTERSHEET_REFS}" (id 0) (at 98.8324 170.1175 0)
-      (effects (font (size 1 1)) (justify left) hide)
-    )
+  (global_label "DTR" (shape input) (at 93.98 170.18 0) (fields_autoplaced)
+    (effects (font (size 1 1)) (justify left))
+    (property "Intersheet References" "${INTERSHEET_REFS}" (id 0) (at 98.6419 170.1175 0)
+      (effects (font (size 1 1)) (justify left) hide)
+    )
